File: kicad/watch/watch.sch (KiCad schematic (older format))
At the start: 36 parts, among them J1 USB_C_Receptacle_USB2.0, J2 Conn_01x04_Female, J3 Conn_01x04_Female, J4 Memory LCD, J5 LCD Frontlight, Q1 Q_NMOS_GDS, SW1 SW_Push, SW2 SW_Push, U1 E73-2G4M08S1C-52840, U2 MCP73831-2-OT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

Commit message: Second rev of schematic. Not yet routed.
Parts:
- removed D1, D2: D_Schottky, Diode_SMD:D_0603_1608Metric_Pad1.05x0.95mm_HandSolder, symbol Device:D_Schottky
- removed U1: E73-2G4M08S1C-52840, nrfmicro:E73-2G4M08S1C-52840, symbol nrfmicro:E73-2G4M08S1C-52840
- removed U3: DS1302S+, Package_SO:SO-8_5.3x6.2mm_P1.27mm, symbol Timer_RTC:DS1302S+
- added D1: D_Schottky_x2_KCom_AAK, Package_TO_SOT_SMD:SOT-23, symbol Device:D_Schottky_x2_KCom_AAK
- added IC1: 113990582, 113990582:113990582, symbol MDBT50Q:113990582
- added J6: Buzzer, Connector_PinHeader_1.00mm:PinHeader_1x02_P1.00mm_Vertical, symbol Connector:Conn_01x02_Female
- added Q2: Q_NMOS_GDS, Package_TO_SOT_SMD:SOT-23, symbol Device:Q_NMOS_GDS
- added R11, R12: R, Resistor_SMD:R_0603_1608Metric_Pad1.05x0.95mm_HandSolder, symbol Device:R
- added U1: W25X20CLUXIG, libs:8-USON, symbol Memory_Flash:AT25SF081-XMHF-X
- added U3: M41T62Q, Package_DFN_QFN:VQFN-16-1EP_3x3mm_P0.5mm_EP1.8x1.8mm, symbol Timer_RTC:M41T62Q
Connections:
- net labels added: BUZZER, FLASH_CLK, FLASH_CS, FLASH_DI, FLASH_DO, RTC_IRQ, SCL, SDA, SQW
- net labels removed: CHRG_STAT, RTC_CLK, RTC_CS, RTC_IO
- wire segments 163 -> 191
- no-connect marks 18 -> 29

Commit message: routed board rev2
Parts:
- added TP10, TP11, TP12, TP13, TP5, TP6, TP7, TP8, TP9: TestPoint, TestPoint:TestPoint_Pad_D1.0mm, symbol Connector:TestPoint
- BT1: footprint Connector_PinSocket_2.00mm:PinSocket_1x02_P2.00mm_Vertical -> Connector_JST:JST_SH_SM02B-SRSS-TB_1x02-1MP_P1.00mm_Horizontal
- J2, J3: footprint Connector_FFC-FPC:Molex_200528-0040_1x04-1MP_P1.00mm_Horizontal -> Connector_JST:JST_SH_SM04B-SRSS-TB_1x04-1MP_P1.00mm_Horizontal
- Q1, Q2: value Q_NMOS_GDS -> DMN6140L; symbol Device:Q_NMOS_GDS -> Device:Q_NMOS_GSD
- TP1, TP2, TP3, TP4: footprint TestPoint:TestPoint_Pad_D1.5mm -> TestPoint:TestPoint_Pad_D1.0mm
Connections:
- net labels removed: EXTCOMIN
- wire segments 191 -> 202
- no-connect marks 29 -> 31
Changed lines of the file:
@@
 F 0 "BT1" H 4568 1546 50  0000 L CNN
 F 1 "Battery_Cell" H 4568 1455 50  0000 L CNN
-F 2 "Connector_PinSocket_2.00mm:PinSocket_1x02_P2.00mm_Vertical" V 4450 1510 50  0001 C CNN
+F 2 "Connector_JST:JST_SH_SM02B-SRSS-TB_1x02-1MP_P1.00mm_Horizontal" V 4450 1510 50  0001 C CNN
 F 3 "~" V 4450 1510 50  0001 C CNN
 	1    4450 1450
@@
 $EndComp
 $Comp
-L Device:Q_NMOS_GDS Q1
+L Device:Q_NMOS_GSD Q1
 U 1 1 5E4FBBEA
 P 10300 5850
 F 0 "Q1" H 10505 5896 50  0000 L CNN
-F 1 "Q_NMOS_GDS" H 10505 5805 50  0000 L CNN
+F 1 "DMN6140L" H 10505 5805 50  0000 L CNN
 F 2 "Package_TO_SOT_SMD:SOT-23" H 10500 5950 50  0001 C CNN
 F 3 "~" H 10300 5850 50  0001 C CNN
@@
 Text GLabel 1000 5100 0    50   Input ~ 0
 LCD_CS
-Text GLabel 1000 5200 0    50   Input ~ 0
-EXTCOMIN
 $Comp
 L Connector:Conn_01x04_Female J2
@@
 F 0 "J2" H 1327 3626 50  0000 L CNN
 F 1 "Conn_01x04_Female" H 1327 3535 50  0000 L CNN
-F 2 "Connector_FFC-FPC:Molex_200528-0040_1x04-1MP_P1.00mm_Horizontal" H 1300 3650 50  0001 C CNN
+F 2 "Connector_JST:JST_SH_SM04B-SRSS-TB_1x04-1MP_P1.00mm_Horizontal" H 1300 3650 50  0001 C CNN
 F 3 "~" H 1300 3650 50  0001 C CNN
 	1    1300 3650
@@
 F 0 "J3" H 2727 3626 50  0000 L CNN
 F 1 "Conn_01x04_Female" H 2727 3535 50  0000 L CNN
-F 2 "Connector_FFC-FPC:Molex_200528-0040_1x04-1MP_P1.00mm_Horizontal" H 2700 3650 50  0001 C CNN
+F 2 "Connector_JST:JST_SH_SM04B-SRSS-TB_1x04-1MP_P1.00mm_Horizontal" H 2700 3650 50  0001 C CNN
 F 3 "~" H 2700 3650 50  0001 C CNN
 	1    2700 3650
@@
 Text GLabel 1000 5600 0    50   Input ~ 0
 BTN2
-Text GLabel 1000 5500 0    50   Input ~ 0
+Text GLabel 1000 5400 0    50   Input ~ 0
 BTN3
-Text GLabel 2950 5800 2    50   Input ~ 0
+Text GLabel 1050 7400 0    50   Input ~ 0
 BTN4
-Text GLabel 2950 5900 2    50   Input ~ 0
+Text GLabel 1050 7200 0    50   Input ~ 0
 BTN5
-Text GLabel 2950 6000 2    50   Input ~ 0
+Text GLabel 1050 7100 0    50   Input ~ 0
 BTN6
 $Comp
@@
 F 0 "TP1" H 3592 3677 50  0000 R CNN
 F 1 "TestPoint" H 3592 3768 50  0000 R CNN
-F 2 "TestPoint:TestPoint_Pad_D1.5mm" H 3850 3650 50  0001 C CNN
+F 2 "TestPoint:TestPoint_Pad_D1.0mm" H 3850 3650 50  0001 C CNN
 F 3 "~" H 3850 3650 50  0001 C CNN
 	1    3650 3650
@@
 F 0 "TP2" H 3708 4170 50  0000 L CNN
 F 1 "TestPoint" H 3708 4079 50  0000 L CNN
-F 2 "TestPoint:TestPoint_Pad_D1.5mm" H 3850 4050 50  0001 C CNN
+F 2 "TestPoint:TestPoint_Pad_D1.0mm" H 3850 4050 50  0001 C CNN
 F 3 "~" H 3850 4050 50  0001 C CNN
 	1    3650 4050
@@
 F 0 "TP3" V 4654 3738 50  0000 L CNN
 F 1 "TestPoint" V 4745 3738 50  0000 L CNN
-F 2 "TestPoint:TestPoint_Pad_D1.5mm" H 4900 3550 50  0001 C CNN
+F 2 "TestPoint:TestPoint_Pad_D1.0mm" H 4900 3550 50  0001 C CNN
 F 3 "~" H 4900 3550 50  0001 C CNN
 	1    4700 3550
@@
 F 0 "TP4" V 4654 4188 50  0000 L CNN
 F 1 "TestPoint" V 4745 4188 50  0000 L CNN
-F 2 "TestPoint:TestPoint_Pad_D1.5mm" H 4900 4000 50  0001 C CNN
+F 2 "TestPoint:TestPoint_Pad_D1.0mm" H 4900 4000 50  0001 C CNN
 F 3 "~" H 4900 4000 50  0001 C CNN
 	1    4700 4000
@@
 Wire Wire Line
 	1100 5100 1000 5100
-Wire Wire Line
-	1100 5200 1000 5200
 Text GLabel 10000 4200 0    50   Input ~ 0
 EXTMODE
@@
 Wire Wire Line
 	3000 5400 2800 5400
-Wire Wire Line
-	1000 5500 1100 5500
 Wire Wire Line
 	1100 5600 1000 5600
@@
 $EndComp
 $Comp
-L Device:Q_NMOS_GDS Q2
+L Device:Q_NMOS_GSD Q2
 U 1 1 5E978039
 P 9250 5850
 F 0 "Q2" H 9455 5896 50  0000 L CNN
-F 1 "Q_NMOS_GDS" H 9455 5805 50  0000 L CNN
+F 1 "DMN6140L" H 9455 5805 50  0000 L CNN
 F 2 "Package_TO_SOT_SMD:SOT-23" H 9450 5950 50  0001 C CNN
 F 3 "~" H 9250 5850 50  0001 C CNN
@@
 	1    0    0    -1
 $EndComp
-Text GLabel 6000 5700 0    50   Input ~ 0
-FLASH_CS
-Text GLabel 6000 5600 0    50   Input ~ 0
-FLASH_CLK
 Text GLabel 7450 5500 2    50   Input ~ 0
 FLASH_DO
-Wire Wire Line
-	6000 5700 6150 5700
-Wire Wire Line
-	6150 5600 6000 5600
-Text GLabel 6000 5500 0    50   Input ~ 0
-FLASH_DI
-Wire Wire Line
-	6000 5500 6150 5500
 Wire Wire Line
 	7350 5500 7450 5500
@@
 Wire Wire Line
 	6050 5900 6150 5900
-Text GLabel 2950 6100 2    50   Input ~ 0
+Text GLabel 2950 6300 2    50   Input ~ 0
 FLASH_CS
 Text GLabel 2950 6200 2    50   Input ~ 0
 FLASH_CLK
-Text GLabel 2950 6300 2    50   Input ~ 0
+Text GLabel 2950 6100 2    50   Input ~ 0
 FLASH_DI
 Wire Wire Line
@@
 Wire Wire Line
 	2950 7000 2800 7000
-NoConn ~ 1100 5400
 NoConn ~ 1100 5800
 NoConn ~ 1100 5900
@@
 NoConn ~ 1100 6500
 NoConn ~ 1100 7000
-NoConn ~ 1100 7100
-NoConn ~ 1100 7200
-NoConn ~ 1100 7400
 NoConn ~ 2800 7500
 NoConn ~ 2800 7400
@@
 	6950 4550 6950 4450
 NoConn ~ 7050 4450
-Text GLabel 7450 4150 2    50   Input ~ 0
+Text GLabel 7500 4600 0    50   Input ~ 0
 SQW
 Wire Wire Line
 	7450 4150 7350 4150
-Text GLabel 7450 4050 2    50   Input ~ 0
+Text GLabel 7500 4700 0    50   Input ~ 0
 RTC_IRQ
 Wire Wire Line
@@
 NoConn ~ 2800 7300
 NoConn ~ 2800 7200
+Text GLabel 1000 6900 0    50   Input ~ 0
+SQW
+Wire Wire Line
+	1000 6900 1100 6900
+$Comp
+L Device:D_Schottky_x2_KCom_AAK D1
+U 1 1 5EC555E3
+P 6250 1350
+F 0 "D1" V 6296 1430 50  0000 L CNN
+F 1 "D_Schottky_x2_KCom_AAK" V 6205 1430 50  0000 L CNN
+F 2 "Package_TO_SOT_SMD:SOT-23" H 6250 1350 50  0001 C CNN
+F 3 "~" H 6250 1350 50  0001 C CNN
+	1    6250 1350
+	0    -1   -1   0
+$EndComp
+Wire Wire Line
+	6550 1000 6550 1350
+Wire Wire Line
+	5400 1650 6250 1650
+Wire Wire Line
+	6450 1350 6550 1350
+$Comp
+L Connector:TestPoint TP9
+U 1 1 5EC78F7F
+P 8050 6100
+F 0 "TP9" V 8004 6288 50  0000 L CNN
+F 1 "TestPoint" V 8095 6288 50  0000 L CNN
+F 2 "TestPoint:TestPoint_Pad_D1.0mm" H 8250 6100 50  0001 C CNN
+F 3 "~" H 8250 6100 50  0001 C CNN
+	1    8050 6100
+	0    1    1    0
+$EndComp
+Text GLabel 7850 6300 0    50   Input ~ 0
+FLASH_CS
+Text GLabel 7850 6200 0    50   Input ~ 0
+FLASH_CLK
+Text GLabel 7850 6100 0    50   Input ~ 0
+FLASH_DI
+Wire Wire Line
+	7850 6100 8050 6100
+$Comp
+L Connector:TestPoint TP10
+U 1 1 5EC96AE2
+P 8050 6200
+F 0 "TP10" V 8004 6388 50  0000 L CNN
+F 1 "TestPoint" V 8095 6388 50  0000 L CNN
+F 2 "TestPoint:TestPoint_Pad_D1.0mm" H 8250 6200 50  0001 C CNN
+F 3 "~" H 8250 6200 50  0001 C CNN
+	1    8050 6200
+	0    1    1    0
+$EndComp
+$Comp
+L Connector:TestPoint TP11
+U 1 1 5ECA09E6
+P 8050 6300
+F 0 "TP11" V 8004 6488 50  0000 L CNN
+F 1 "TestPoint" V 8095 6488 50  0000 L CNN
+F 2 "TestPoint:TestPoint_Pad_D1.0mm" H 8250 6300 50  0001 C CNN
+F 3 "~" H 8250 6300 50  0001 C CNN
+	1    8050 6300
+	0    1    1    0
+$EndComp
+Wire Wire Line
+	7850 6200 8050 6200
+Wire Wire Line
+	7850 6300 8050 6300
+Text GLabel 7850 6400 0    50   Input ~ 0
+FLASH_DO
+$Comp
+L Connector:TestPoint TP12
+U 1 1 5ECB4CB4
+P 8050 6400
+F 0 "TP12" V 8004 6588 50  0000 L CNN
+F 1 "TestPoint" V 8095 6588 50  0000 L CNN
+F 2 "TestPoint:TestPoint_Pad_D1.0mm" H 8250 6400 50  0001 C CNN
+F 3 "~" H 8250 6400 50  0001 C CNN
+	1    8050 6400
+	0    1    1    0
+$EndComp
+Wire Wire Line
+	8050 6400 7850 6400
+$Comp
+L Connector:TestPoint TP5
+U 1 1 5ECC4057
+P 7650 4400
+F 0 "TP5" V 7604 4588 50  0000 L CNN
+F 1 "TestPoint" V 7695 4588 50  0000 L CNN
+F 2 "TestPoint:TestPoint_Pad_D1.0mm" H 7850 4400 50  0001 C CNN
+F 3 "~" H 7850 4400 50  0001 C CNN
+	1    7650 4400
+	0    1    1    0
+$EndComp
+$Comp
+L Connector:TestPoint TP6
+U 1 1 5ECC405D
+P 7650 4500
+F 0 "TP6" V 7604 4688 50  0000 L CNN
+F 1 "TestPoint" V 7695 4688 50  0000 L CNN
+F 2 "TestPoint:TestPoint_Pad_D1.0mm" H 7850 4500 50  0001 C CNN
+F 3 "~" H 7850 4500 50  0001 C CNN
+	1    7650 4500
+	0    1    1    0
+$EndComp
+$Comp
+L Connector:TestPoint TP7
+U 1 1 5ECC4063
+P 7650 4600
+F 0 "TP7" V 7604 4788 50  0000 L CNN
+F 1 "TestPoint" V 7695 4788 50  0000 L CNN
+F 2 "TestPoint:TestPoint_Pad_D1.0mm" H 7850 4600 50  0001 C CNN
+F 3 "~" H 7850 4600 50  0001 C CNN
+	1    7650 4600
+	0    1    1    0
+$EndComp
+$Comp
+L Connector:TestPoint TP8
+U 1 1 5ECC4069
+P 7650 4700
+F 0 "TP8" V 7604 4888 50  0000 L CNN
+F 1 "TestPoint" V 7695 4888 50  0000 L CNN
+F 2 "TestPoint:TestPoint_Pad_D1.0mm" H 7850 4700 50  0001 C CNN
+F 3 "~" H 7850 4700 50  0001 C CNN
+	1    7650 4700
+	0    1    1    0
+$EndComp
+Text GLabel 7500 4400 0    50   Input ~ 0
+SCL
+Text GLabel 7500 4500 0    50   Input ~ 0
+SDA
+Wire Wire Line
+	7500 4600 7650 4600
+Wire Wire Line
+	7500 4500 7650 4500
+Wire Wire Line
+	7500 4400 7650 4400
+Wire Wire Line
+	7650 4700 7500 4700
+Text GLabel 8000 2000 0    50   Input ~ 0
+VIN
+$Comp
+L Connector:TestPoint TP13
+U 1 1 5ED26D0C
+P 8100 2000
+F 0 "TP13" V 8054 2188 50  0000 L CNN
+F 1 "TestPoint" V 8145 2188 50  0000 L CNN
+F 2 "TestPoint:TestPoint_Pad_D1.0mm" H 8300 2000 50  0001 C CNN
+F 3 "~" H 8300 2000 50  0001 C CNN
+	1    8100 2000
+	0    1    1    0
+$EndComp
+Wire Wire Line
+	8100 2000 8000 2000
+Text GLabel 6050 5700 0    50   Input ~ 0
+FLASH_CS
+Text GLabel 6050 5600 0    50   Input ~ 0
+FLASH_CLK
+Text GLabel 6050 5500 0    50   Input ~ 0
+FLASH_DI
+Wire Wire Line
+	6050 5500 6150 5500
+Wire Wire Line
+	6150 5600 6050 5600
+Wire Wire Line
+	6050 5700 6150 5700
+Text GLabel 7450 4150 2    50   Input ~ 0
+SQW
+Text GLabel 7450 4050 2    50   Input ~ 0
+RTC_IRQ
+NoConn ~ 1100 5200
+Wire Wire Line
+	1000 5400 1100 5400
+NoConn ~ 1100 5500
 $Comp
 L MDBT50Q:113990582 IC1
@@
 	1    0    0    -1
 $EndComp
-Text GLabel 1000 6900 0    50   Input ~ 0
-SQW
-Wire Wire Line
-	1000 6900 1100 6900
-$Comp
-L Device:D_Schottky_x2_KCom_AAK D1
-U 1 1 5EC555E3
-P 6250 1350
-F 0 "D1" V 6296 1430 50  0000 L CNN
-F 1 "D_Schottky_x2_KCom_AAK" V 6205 1430 50  0000 L CNN
-F 2 "Package_TO_SOT_SMD:SOT-23" H 6250 1350 50  0001 C CNN
-F 3 "~" H 6250 1350 50  0001 C CNN
-	1    6250 1350
-	0    -1   -1   0
-$EndComp
-Wire Wire Line
-	6550 1000 6550 1350
-Wire Wire Line
-	5400 1650 6250 1650
-Wire Wire Line
-	6450 1350 6550 1350
+Wire Wire Line
+	1050 7400 1100 7400
+Wire Wire Line
+	1100 7200 1050 7200
+Wire Wire Line
+	1100 7100 1050 7100
+NoConn ~ 2950 5800
+NoConn ~ 2950 5900
+NoConn ~ 2950 6000
+NoConn ~ 2800 4300
 $EndSCHEMATC

Commit message: added voltage divider for battery reading
Parts:
- added R13: 2M, Resistor_SMD:R_0603_1608Metric_Pad1.05x0.95mm_HandSolder, symbol Device:R
- added R14: 4M, Resistor_SMD:R_0603_1608Metric_Pad1.05x0.95mm_HandSolder, symbol Device:R
Connections:
- net labels added: BATREAD
- wire segments 202 -> 208
- no-connect marks 31 -> 29
Changed lines of the file:
@@
 NoConn ~ 1100 6100
 NoConn ~ 1100 6400
-NoConn ~ 1100 6500
 NoConn ~ 1100 7000
 NoConn ~ 2800 7500
@@
 NoConn ~ 2950 5900
 NoConn ~ 2950 6000
-NoConn ~ 2800 4300
+Text GLabel 1000 6500 0    50   Input ~ 0
+BATREAD
+Wire Wire Line
+	1000 6500 1100 6500
+$Comp
+L power:+BATT #PWR0142
+U 1 1 5EE2B5E9
+P 4250 5100
+F 0 "#PWR0142" H 4250 4950 50  0001 C CNN
+F 1 "+BATT" H 4265 5273 50  0000 C CNN
+F 2 "" H 4250 5100 50  0001 C CNN
+F 3 "" H 4250 5100 50  0001 C CNN
+	1    4250 5100
+	1    0    0    -1
+$EndComp
+$Comp
+L Device:R R13
+U 1 1 5EE2B715
+P 4250 5300
+F 0 "R13" H 4320 5346 50  0000 L CNN
+F 1 "2M" H 4320 5255 50  0000 L CNN
+F 2 "Resistor_SMD:R_0603_1608Metric_Pad1.05x0.95mm_HandSolder" V 4180 5300 50  0001 C CNN
+F 3 "~" H 4250 5300 50  0001 C CNN
+	1    4250 5300
+	1    0    0    -1
+$EndComp
+Wire Wire Line
+	4250 5100 4250 5150
+$Comp
+L Device:R R14
+U 1 1 5EE37143
+P 4250 5700
+F 0 "R14" H 4320 5746 50  0000 L CNN
+F 1 "4M" H 4320 5655 50  0000 L CNN
+F 2 "Resistor_SMD:R_0603_1608Metric_Pad1.05x0.95mm_HandSolder" V 4180 5700 50  0001 C CNN
+F 3 "~" H 4250 5700 50  0001 C CNN
+	1    4250 5700
+	1    0    0    -1
+$EndComp
+Wire Wire Line
+	4250 5550 4250 5500
+Text GLabel 4400 5500 2    50   Input ~ 0
+BATREAD
+Wire Wire Line
+	4400 5500 4250 5500
+Connection ~ 4250 5500
+Wire Wire Line
+	4250 5500 4250 5450
+$Comp
+L power:GND #PWR0143
+U 1 1 5EE4F9F8
+P 4250 5950
+F 0 "#PWR0143" H 4250 5700 50  0001 C CNN
+F 1 "GND" H 4255 5777 50  0000 C CNN
+F 2 "" H 4250 5950 50  0001 C CNN
+F 3 "" H 4250 5950 50  0001 C CNN
+	1    4250 5950
+	1    0    0    -1
+$EndComp
+Wire Wire Line
+	4250 5950 4250 5850
 $EndSCHEMATC

Commit message: Add qwiic jumpers for accessory ports
Parts:
- added JP1, JP2: Jumper_NO_Small, Jumper:SolderJumper-2_P1.3mm_Open_RoundedPad1.0x1.5mm, symbol Device:Jumper_NO_Small
- added R15, R16: 4k7, Resistor_SMD:R_0603_1608Metric_Pad1.05x0.95mm_HandSolder, symbol Device:R
Connections:
- wire segments 208 -> 217
Changed lines of the file:
@@
 	1    0    0    -1
 $EndComp
-Text GLabel 1000 3550 0    50   Input ~ 0
+Text GLabel 1000 3850 0    50   Input ~ 0
 BTN1
 Wire Wire Line
@@
 L power:GND #PWR0130
 U 1 1 5E55FF3B
-P 1000 3850
-F 0 "#PWR0130" H 1000 3600 50  0001 C CNN
-F 1 "GND" H 1005 3677 50  0000 C CNN
-F 2 "" H 1000 3850 50  0001 C CNN
-F 3 "" H 1000 3850 50  0001 C CNN
-	1    1000 3850
-	1    0    0    -1
-$EndComp
-Wire Wire Line
-	1000 3850 1100 3850
+P 1000 3550
+F 0 "#PWR0130" H 1000 3300 50  0001 C CNN
+F 1 "GND" V 1005 3422 50  0000 R CNN
+F 2 "" H 1000 3550 50  0001 C CNN
+F 3 "" H 1000 3550 50  0001 C CNN
+	1    1000 3550
+	0    1    1    0
+$EndComp
 Wire Wire Line
 	1100 3750 1000 3750
@@
 L Connector:Conn_01x04_Female J3
 U 1 1 5E573B85
-P 2700 3650
-F 0 "J3" H 2727 3626 50  0000 L CNN
-F 1 "Conn_01x04_Female" H 2727 3535 50  0000 L CNN
-F 2 "Connector_JST:JST_SH_SM04B-SRSS-TB_1x04-1MP_P1.00mm_Horizontal" H 2700 3650 50  0001 C CNN
-F 3 "~" H 2700 3650 50  0001 C CNN
-	1    2700 3650
-	1    0    0    -1
-$EndComp
-Text GLabel 2400 3550 0    50   Input ~ 0
+P 2900 3550
+F 0 "J3" H 2927 3526 50  0000 L CNN
+F 1 "Conn_01x04_Female" H 2927 3435 50  0000 L CNN
+F 2 "Connector_JST:JST_SH_SM04B-SRSS-TB_1x04-1MP_P1.00mm_Horizontal" H 2900 3550 50  0001 C CNN
+F 3 "~" H 2900 3550 50  0001 C CNN
+	1    2900 3550
+	1    0    0    -1
+$EndComp
+Text GLabel 2550 3750 0    50   Input ~ 0
 BTN4
-Wire Wire Line
-	2400 3550 2500 3550
-Text GLabel 2400 3650 0    50   Input ~ 0
+Text GLabel 2550 3650 0    50   Input ~ 0
 BTN5
-Text GLabel 2400 3750 0    50   Input ~ 0
-BTN6
 $Comp
 L power:GND #PWR0131
 U 1 1 5E573B8F
-P 2400 3850
-F 0 "#PWR0131" H 2400 3600 50  0001 C CNN
-F 1 "GND" H 2405 3677 50  0000 C CNN
-F 2 "" H 2400 3850 50  0001 C CNN
-F 3 "" H 2400 3850 50  0001 C CNN
-	1    2400 3850
-	1    0    0    -1
-$EndComp
-Wire Wire Line
-	2400 3850 2500 3850
-Wire Wire Line
-	2500 3750 2400 3750
-Wire Wire Line
-	2400 3650 2500 3650
+P 2500 3450
+F 0 "#PWR0131" H 2500 3200 50  0001 C CNN
+F 1 "GND" V 2505 3322 50  0000 R CNN
+F 2 "" H 2500 3450 50  0001 C CNN
+F 3 "" H 2500 3450 50  0001 C CNN
+	1    2500 3450
+	0    1    1    0
+$EndComp
 Text GLabel 2950 5600 2    50   Input ~ 0
 FRONTLIGHT
@@
 Wire Wire Line
 	4250 5950 4250 5850
+$Comp
+L power:+3V3 #PWR0144
+U 1 1 5EE606BF
+P 5300 4600
+F 0 "#PWR0144" H 5300 4450 50  0001 C CNN
+F 1 "+3V3" H 5315 4773 50  0000 C CNN
+F 2 "" H 5300 4600 50  0001 C CNN
+F 3 "" H 5300 4600 50  0001 C CNN
+	1    5300 4600
+	1    0    0    -1
+$EndComp
+$Comp
+L Device:R R15
+U 1 1 5EE6175A
+P 5150 4800
+F 0 "R15" H 5220 4846 50  0000 L CNN
+F 1 "4k7" V 5150 4750 50  0000 L CNN
+F 2 "Resistor_SMD:R_0603_1608Metric_Pad1.05x0.95mm_HandSolder" V 5080 4800 50  0001 C CNN
+F 3 "~" H 5150 4800 50  0001 C CNN
+	1    5150 4800
+	1    0    0    -1
+$EndComp
+$Comp
+L Device:R R16
+U 1 1 5EE618DB
+P 5450 4800
+F 0 "R16" H 5520 4846 50  0000 L CNN
+F 1 "4k7" V 5450 4750 50  0000 L CNN
+F 2 "Resistor_SMD:R_0603_1608Metric_Pad1.05x0.95mm_HandSolder" V 5380 4800 50  0001 C CNN
+F 3 "~" H 5450 4800 50  0001 C CNN
+	1    5450 4800
+	1    0    0    -1
+$EndComp
+Text GLabel 5150 5000 3    50   Input ~ 0
+SDA
+Text GLabel 5450 5000 3    50   Input ~ 0
+SCL
+Wire Wire Line
+	5450 5000 5450 4950
+Wire Wire Line
+	5150 4950 5150 5000
+Wire Wire Line
+	5300 4600 5300 4650
+Wire Wire Line
+	5300 4650 5150 4650
+Wire Wire Line
+	5450 4650 5300 4650
+Connection ~ 5300 4650
+$Comp
+L power:+3V3 #PWR0145
+U 1 1 5EE942BD
+P 2450 3150
+F 0 "#PWR0145" H 2450 3000 50  0001 C CNN
+F 1 "+3V3" V 2465 3278 50  0000 L CNN
+F 2 "" H 2450 3150 50  0001 C CNN
+F 3 "" H 2450 3150 50  0001 C CNN
+	1    2450 3150
+	0    -1   -1   0
+$EndComp
+Wire Wire Line
+	1000 3850 1100 3850
+Wire Wire Line
+	2550 3650 2700 3650
+Wire Wire Line
+	2550 3750 2700 3750
+Wire Wire Line
+	2500 3450 2700 3450
+Text GLabel 2550 3550 0    50   Input ~ 0
+BTN6
+Wire Wire Line
+	2550 3550 2700 3550
+$Comp
+L Device:Jumper_NO_Small JP2
+U 1 1 5EEFF096
+P 2700 4000
+F 0 "JP2" H 2700 4185 50  0000 C CNN
+F 1 "Jumper_NO_Small" H 2700 4094 50  0000 C CNN
+F 2 "Jumper:SolderJumper-2_P1.3mm_Open_RoundedPad1.0x1.5mm" H 2700 4000 50  0001 C CNN
+F 3 "~" H 2700 4000 50  0001 C CNN
+	1    2700 4000
+	1    0    0    -1
+$EndComp
+Text GLabel 2550 4000 0    50   Input ~ 0
+BTN6
+Wire Wire Line
+	2550 4000 2600 4000
+$Comp
+L power:+3V3 #PWR0146
+U 1 1 5EF0C055
+P 2850 4000
+F 0 "#PWR0146" H 2850 3850 50  0001 C CNN
+F 1 "+3V3" V 2865 4128 50  0000 L CNN
+F 2 "" H 2850 4000 50  0001 C CNN
+F 3 "" H 2850 4000 50  0001 C CNN
+	1    2850 4000
+	0    1    1    0
+$EndComp
+Wire Wire Line
+	2850 4000 2800 4000
+$Comp
+L Device:Jumper_NO_Small JP1
+U 1 1 5EF19233
+P 1300 4000
+F 0 "JP1" H 1300 4185 50  0000 C CNN
+F 1 "Jumper_NO_Small" H 1300 4094 50  0000 C CNN
+F 2 "Jumper:SolderJumper-2_P1.3mm_Open_RoundedPad1.0x1.5mm" H 1300 4000 50  0001 C CNN
+F 3 "~" H 1300 4000 50  0001 C CNN
+	1    1300 4000
+	1    0    0    -1
+$EndComp
+Text GLabel 1150 4000 0    50   Input ~ 0
+BTN2
+Wire Wire Line
+	1150 4000 1200 4000
+$Comp
+L power:+3V3 #PWR0147
+U 1 1 5EF1923B
+P 1450 4000
+F 0 "#PWR0147" H 1450 3850 50  0001 C CNN
+F 1 "+3V3" V 1465 4128 50  0000 L CNN
+F 2 "" H 1450 4000 50  0001 C CNN
+F 3 "" H 1450 4000 50  0001 C CNN
+	1    1450 4000
+	0    1    1    0
+$EndComp
+Wire Wire Line
+	1450 4000 1400 4000
 $EndSCHEMATC

Commit message: checkpoint before redoing schematic
Parts:
- R15, R16: value 4k7 -> 5.1k
Changed lines of the file:
@@
 EESchema Schematic File Version 4
+LIBS:watch-cache
 EELAYER 26 0
 EELAYER END
@@
 P 5150 4800
 F 0 "R15" H 5220 4846 50  0000 L CNN
-F 1 "4k7" V 5150 4750 50  0000 L CNN
+F 1 "5.1k" V 5150 4700 50  0000 L CNN
 F 2 "Resistor_SMD:R_0603_1608Metric_Pad1.05x0.95mm_HandSolder" V 5080 4800 50  0001 C CNN
 F 3 "~" H 5150 4800 50  0001 C CNN
@@
 P 5450 4800
 F 0 "R16" H 5520 4846 50  0000 L CNN
-F 1 "4k7" V 5450 4750 50  0000 L CNN
+F 1 "5.1k" V 5450 4700 50  0000 L CNN
 F 2 "Resistor_SMD:R_0603_1608Metric_Pad1.05x0.95mm_HandSolder" V 5380 4800 50  0001 C CNN
 F 3 "~" H 5450 4800 50  0001 C CNN
