File: kicad/watch/watch.sch (KiCad schematic (older format))
At the start: 55 parts, among them IC1 113990582, J1 USB_C_Receptacle_USB2.0, J2 Conn_01x04_Female, J3 Conn_01x04_Female, J4 Memory LCD, J5 LCD Frontlight, J6 Buzzer, Q1 DMN6140L, Q2 DMN6140L, SW1 SW_Push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

Commit message: un-derped pcb references
Parts:
- R15, R16: value 5.1k -> 4k7
- renumbered SW2 to SW_BOOT1, SW1 to SW_RESET1
Changed lines of the file:
@@
 Wire Wire Line
 	2950 2050 2950 1950
+Connection ~ 2950 1950
 Wire Wire Line
 	2950 1950 2650 1950
@@
 BTN6
 $Comp
-L Switch:SW_Push SW1
+L Switch:SW_Push SW_RESET1
 U 1 1 5E5F1A61
 P 4100 7150
-F 0 "SW1" V 4054 7298 50  0000 L CNN
+F 0 "SW_RESET1" V 4054 7298 50  0000 L CNN
 F 1 "SW_Push" V 4145 7298 50  0000 L CNN
 F 2 "Button_Switch_SMD:SW_SPST_CK_KXT3" H 4100 7350 50  0001 C CNN
@@
 BOOTLOAD
 $Comp
-L Switch:SW_Push SW2
+L Switch:SW_Push SW_BOOT1
 U 1 1 5E6211CF
 P 4700 7150
-F 0 "SW2" V 4654 7298 50  0000 L CNN
+F 0 "SW_BOOT1" V 4654 7298 50  0000 L CNN
 F 1 "SW_Push" V 4745 7298 50  0000 L CNN
 F 2 "Button_Switch_SMD:SW_SPST_CK_KXT3" H 4700 7350 50  0001 C CNN
@@
 L Connector:TestPoint TP9
 U 1 1 5EC78F7F
-P 8050 6100
-F 0 "TP9" V 8004 6288 50  0000 L CNN
-F 1 "TestPoint" V 8095 6288 50  0000 L CNN
-F 2 "TestPoint:TestPoint_Pad_D1.0mm" H 8250 6100 50  0001 C CNN
-F 3 "~" H 8250 6100 50  0001 C CNN
-	1    8050 6100
-	0    1    1    0
-$EndComp
-Text GLabel 7850 6300 0    50   Input ~ 0
+P 8050 6000
+F 0 "TP9" V 8004 6188 50  0000 L CNN
+F 1 "TestPoint" V 8095 6188 50  0000 L CNN
+F 2 "TestPoint:TestPoint_Pad_D1.0mm" H 8250 6000 50  0001 C CNN
+F 3 "~" H 8250 6000 50  0001 C CNN
+	1    8050 6000
+	0    1    1    0
+$EndComp
+Text GLabel 7850 6400 0    50   Input ~ 0
 FLASH_CS
 Text GLabel 7850 6200 0    50   Input ~ 0
 FLASH_CLK
-Text GLabel 7850 6100 0    50   Input ~ 0
+Text GLabel 7850 6000 0    50   Input ~ 0
 FLASH_DI
 Wire Wire Line
-	7850 6100 8050 6100
+	7850 6000 8050 6000
 $Comp
 L Connector:TestPoint TP10
@@
 L Connector:TestPoint TP11
 U 1 1 5ECA09E6
-P 8050 6300
-F 0 "TP11" V 8004 6488 50  0000 L CNN
-F 1 "TestPoint" V 8095 6488 50  0000 L CNN
-F 2 "TestPoint:TestPoint_Pad_D1.0mm" H 8250 6300 50  0001 C CNN
-F 3 "~" H 8250 6300 50  0001 C CNN
-	1    8050 6300
-	0    1    1    0
-$EndComp
-Wire Wire Line
-	7850 6200 8050 6200
-Wire Wire Line
-	7850 6300 8050 6300
-Text GLabel 7850 6400 0    50   Input ~ 0
-FLASH_DO
-$Comp
-L Connector:TestPoint TP12
-U 1 1 5ECB4CB4
 P 8050 6400
-F 0 "TP12" V 8004 6588 50  0000 L CNN
+F 0 "TP11" V 8004 6588 50  0000 L CNN
 F 1 "TestPoint" V 8095 6588 50  0000 L CNN
 F 2 "TestPoint:TestPoint_Pad_D1.0mm" H 8250 6400 50  0001 C CNN
@@
 $EndComp
 Wire Wire Line
-	8050 6400 7850 6400
+	7850 6200 8050 6200
+Wire Wire Line
+	7850 6400 8050 6400
+Text GLabel 7850 6600 0    50   Input ~ 0
+FLASH_DO
+$Comp
+L Connector:TestPoint TP12
+U 1 1 5ECB4CB4
+P 8050 6600
+F 0 "TP12" V 8004 6788 50  0000 L CNN
+F 1 "TestPoint" V 8095 6788 50  0000 L CNN
+F 2 "TestPoint:TestPoint_Pad_D1.0mm" H 8250 6600 50  0001 C CNN
+F 3 "~" H 8250 6600 50  0001 C CNN
+	1    8050 6600
+	0    1    1    0
+$EndComp
+Wire Wire Line
+	8050 6600 7850 6600
 $Comp
 L Connector:TestPoint TP5
@@
 P 7650 4400
 F 0 "TP5" V 7604 4588 50  0000 L CNN
-F 1 "TestPoint" V 7695 4588 50  0000 L CNN
+F 1 "TestPoint" V 7650 4850 50  0000 L CNN
 F 2 "TestPoint:TestPoint_Pad_D1.0mm" H 7850 4400 50  0001 C CNN
 F 3 "~" H 7850 4400 50  0001 C CNN
@@
 P 7650 4500
 F 0 "TP6" V 7604 4688 50  0000 L CNN
-F 1 "TestPoint" V 7695 4688 50  0000 L CNN
+F 1 "TestPoint" V 7650 5000 50  0000 L CNN
 F 2 "TestPoint:TestPoint_Pad_D1.0mm" H 7850 4500 50  0001 C CNN
 F 3 "~" H 7850 4500 50  0001 C CNN
@@
 P 7650 4600
 F 0 "TP7" V 7604 4788 50  0000 L CNN
-F 1 "TestPoint" V 7695 4788 50  0000 L CNN
+F 1 "TestPoint" V 7650 5050 50  0000 L CNN
 F 2 "TestPoint:TestPoint_Pad_D1.0mm" H 7850 4600 50  0001 C CNN
 F 3 "~" H 7850 4600 50  0001 C CNN
@@
 P 7650 4700
 F 0 "TP8" V 7604 4888 50  0000 L CNN
-F 1 "TestPoint" V 7695 4888 50  0000 L CNN
+F 1 "TestPoint" V 7600 5150 50  0000 L CNN
 F 2 "TestPoint:TestPoint_Pad_D1.0mm" H 7850 4700 50  0001 C CNN
 F 3 "~" H 7850 4700 50  0001 C CNN
@@
 P 5150 4800
 F 0 "R15" H 5220 4846 50  0000 L CNN
-F 1 "5.1k" V 5150 4700 50  0000 L CNN
+F 1 "4k7" V 5150 4750 50  0000 L CNN
 F 2 "Resistor_SMD:R_0603_1608Metric_Pad1.05x0.95mm_HandSolder" V 5080 4800 50  0001 C CNN
 F 3 "~" H 5150 4800 50  0001 C CNN
@@
 P 5450 4800
 F 0 "R16" H 5520 4846 50  0000 L CNN
-F 1 "5.1k" V 5450 4700 50  0000 L CNN
+F 1 "4k7" V 5450 4750 50  0000 L CNN
 F 2 "Resistor_SMD:R_0603_1608Metric_Pad1.05x0.95mm_HandSolder" V 5380 4800 50  0001 C CNN
 F 3 "~" H 5450 4800 50  0001 C CNN
@@
 Wire Wire Line
 	1450 4000 1400 4000
-Connection ~ 2950 1950
 $EndSCHEMATC

Commit message: checkpoint before retooling board...again.
Parts:
- removed J1: USB_C_Receptacle_USB2.0, Connector_USB:USB_C_Receptacle_Palconn_UTC16-G, symbol Connector:USB_C_Receptacle_USB2.0
- removed R1, R2: 5.1k, Resistor_SMD:R_0603_1608Metric_Pad1.05x0.95mm_HandSolder, symbol Device:R
- added J1: Conn_01x04_Female, Connector_JST:JST_SH_SM04B-SRSS-TB_1x04-1MP_P1.00mm_Horizontal, symbol Connector:Conn_01x04_Female
Connections:
- wire segments 217 -> 203
- no-connect marks 29 -> 27
Other:
- note removed: "USB-C Port (legacy USB mode)"
Changed lines of the file:
@@
 $EndDescr
-$Comp
-L Connector:USB_C_Receptacle_USB2.0 J1
-U 1 1 5E43554D
-P 950 1550
-F 0 "J1" H 1055 2417 50  0000 C CNN
-F 1 "USB_C_Receptacle_USB2.0" H 1055 2326 50  0000 C CNN
-F 2 "Connector_USB:USB_C_Receptacle_Palconn_UTC16-G" H 1100 1550 50  0001 C CNN
-F 3 "https://www.usb.org/sites/default/files/documents/usb_type-c.zip" H 1100 1550 50  0001 C CNN
-	1    950  1550
-	1    0    0    -1
-$EndComp
-NoConn ~ 1550 2050
-NoConn ~ 1550 2150
 $Comp
 L power:VBUS #PWR0105
 U 1 1 5E4357E3
-P 1800 750
-F 0 "#PWR0105" H 1800 600 50  0001 C CNN
-F 1 "VBUS" H 1815 923 50  0000 C CNN
-F 2 "" H 1800 750 50  0001 C CNN
-F 3 "" H 1800 750 50  0001 C CNN
-	1    1800 750
-	1    0    0    -1
-$EndComp
-Wire Wire Line
-	1800 750  1800 950
-Wire Wire Line
-	1800 950  1550 950
-$Comp
-L Device:R R2
-U 1 1 5E43586A
-P 1850 1250
-F 0 "R2" V 1900 1100 50  0000 C CNN
-F 1 "5.1k" V 1850 1250 50  0000 C CNN
-F 2 "Resistor_SMD:R_0603_1608Metric_Pad1.05x0.95mm_HandSolder" V 1780 1250 50  0001 C CNN
-F 3 "~" H 1850 1250 50  0001 C CNN
-	1    1850 1250
-	0    1    1    0
-$EndComp
-Wire Wire Line
-	1550 1250 1700 1250
-$Comp
-L Device:R R1
-U 1 1 5E43595E
-P 1850 1150
-F 0 "R1" V 1800 1000 50  0000 C CNN
-F 1 "5.1k" V 1850 1150 50  0000 C CNN
-F 2 "Resistor_SMD:R_0603_1608Metric_Pad1.05x0.95mm_HandSolder" V 1780 1150 50  0001 C CNN
-F 3 "~" H 1850 1150 50  0001 C CNN
-	1    1850 1150
-	0    1    1    0
-$EndComp
-Wire Wire Line
-	1550 1150 1700 1150
-$Comp
-L power:GND #PWR0106
-U 1 1 5E435A38
-P 2200 1350
-F 0 "#PWR0106" H 2200 1100 50  0001 C CNN
-F 1 "GND" H 2205 1177 50  0000 C CNN
-F 2 "" H 2200 1350 50  0001 C CNN
-F 3 "" H 2200 1350 50  0001 C CNN
-	1    2200 1350
-	1    0    0    -1
-$EndComp
-Wire Wire Line
-	2200 1350 2200 1250
-Wire Wire Line
-	2200 1150 2000 1150
-Wire Wire Line
-	2000 1250 2200 1250
-Connection ~ 2200 1250
-Wire Wire Line
-	2200 1250 2200 1150
-Wire Wire Line
-	1550 1450 1650 1450
-Wire Wire Line
-	1550 1550 1650 1550
-Wire Wire Line
-	1650 1550 1650 1450
-Wire Wire Line
-	1550 1750 1650 1750
-Wire Wire Line
-	1550 1650 1650 1650
-Wire Wire Line
-	1650 1650 1650 1750
-$Comp
-L power:GND #PWR0107
-U 1 1 5E43601B
-P 950 2650
-F 0 "#PWR0107" H 950 2400 50  0001 C CNN
-F 1 "GND" H 955 2477 50  0000 C CNN
-F 2 "" H 950 2650 50  0001 C CNN
-F 3 "" H 950 2650 50  0001 C CNN
-	1    950  2650
-	1    0    0    -1
-$EndComp
-Wire Wire Line
-	950  2650 950  2550
-Wire Wire Line
-	650  2450 650  2550
-Wire Wire Line
-	650  2550 950  2550
-Connection ~ 950  2550
-Wire Wire Line
-	950  2550 950  2450
+P 1400 1400
+F 0 "#PWR0105" H 1400 1250 50  0001 C CNN
+F 1 "VBUS" H 1415 1573 50  0000 C CNN
+F 2 "" H 1400 1400 50  0001 C CNN
+F 3 "" H 1400 1400 50  0001 C CNN
+	1    1400 1400
+	1    0    0    -1
+$EndComp
 $Comp
 L Battery_Management:MCP73831-2-OT U2
@@
 Wire Wire Line
 	7250 2050 7250 1900
-Text Notes 1200 2400 0    50   ~ 0
-USB-C Port (legacy USB mode)
 Text Notes 3350 1800 0    50   ~ 0
 Battery charger IC
@@
 Text GLabel 3300 4800 2    50   Input ~ 0
 USB_DN
-Text GLabel 1750 1750 2    50   Input ~ 0
+Text GLabel 1400 1700 2    50   Input ~ 0
 USB_DP
-Wire Wire Line
-	1750 1750 1650 1750
-Connection ~ 1650 1750
-Text GLabel 1750 1550 2    50   Input ~ 0
+Text GLabel 1400 1600 2    50   Input ~ 0
 USB_DN
-Wire Wire Line
-	1750 1550 1650 1550
-Connection ~ 1650 1550
 Text GLabel 6700 1000 2    50   Input ~ 0
 VIN
@@
 	5450 4650 5300 4650
 Connection ~ 5300 4650
-$Comp
-L power:+3V3 #PWR0145
-U 1 1 5EE942BD
-P 2450 3150
-F 0 "#PWR0145" H 2450 3000 50  0001 C CNN
-F 1 "+3V3" V 2465 3278 50  0000 L CNN
-F 2 "" H 2450 3150 50  0001 C CNN
-F 3 "" H 2450 3150 50  0001 C CNN
-	1    2450 3150
-	0    -1   -1   0
-$EndComp
 Wire Wire Line
 	1000 3850 1100 3850
@@
 Wire Wire Line
 	1450 4000 1400 4000
+$Comp
+L Connector:Conn_01x04_Female J1
+U 1 1 5E541D8B
+P 1100 1700
+F 0 "J1" H 1127 1676 50  0000 L CNN
+F 1 "Conn_01x04_Female" H 1127 1585 50  0000 L CNN
+F 2 "Connector_JST:JST_SH_SM04B-SRSS-TB_1x04-1MP_P1.00mm_Horizontal" H 1100 1700 50  0001 C CNN
+F 3 "~" H 1100 1700 50  0001 C CNN
+	1    1100 1700
+	-1   0    0    1
+$EndComp
+Wire Wire Line
+	1400 1400 1400 1500
+Wire Wire Line
+	1400 1500 1300 1500
+Wire Wire Line
+	1400 1600 1300 1600
+Wire Wire Line
+	1400 1700 1300 1700
+$Comp
+L power:GND #PWR0106
+U 1 1 5E5661C7
+P 1400 1850
+F 0 "#PWR0106" H 1400 1600 50  0001 C CNN
+F 1 "GND" H 1405 1677 50  0000 C CNN
+F 2 "" H 1400 1850 50  0001 C CNN
+F 3 "" H 1400 1850 50  0001 C CNN
+	1    1400 1850
+	1    0    0    -1
+$EndComp
+Wire Wire Line
+	1400 1850 1400 1800
+Wire Wire Line
+	1400 1800 1300 1800
 $EndSCHEMATC

Commit message: checkpoint
Parts:
- removed R13: 2M, Resistor_SMD:R_0603_1608Metric_Pad1.05x0.95mm_HandSolder, symbol Device:R
- removed R14: 4M, Resistor_SMD:R_0603_1608Metric_Pad1.05x0.95mm_HandSolder, symbol Device:R
- removed U3: M41T62Q, Package_DFN_QFN:VQFN-16-1EP_3x3mm_P0.5mm_EP1.8x1.8mm, symbol Timer_RTC:M41T62Q
- removed Y2: 32.768 kHz, Crystal:Crystal_SMD_2012-2Pin_2.0x1.2mm_HandSoldering, symbol Device:Crystal
- added C5: 11mF, Capacitor_SMD:C_1210_3225Metric_Pad1.42x2.65mm_HandSolder, symbol Device:C
- added C6: 4.7 uF, Capacitor_SMD:C_0603_1608Metric_Pad1.05x0.95mm_HandSolder, symbol Device:C
- added D2: D_Schottky, Diode_SMD:D_SOT-23_ANK, symbol Device:D_Schottky
- added IC2: M41T62LC6F, libs:LCC90P230X50X80-8N, symbol M41T62LC6F:M41T62LC6F
- added JP3: Jumper_NO_Small, Jumper:SolderJumper-2_P1.3mm_Open_RoundedPad1.0x1.5mm, symbol Device:Jumper_NO_Small
- added L2: 4.7 uH, Inductor_SMD:L_0603_1608Metric_Pad1.05x0.95mm_HandSolder, symbol Device:L
- added R1: 10 m, Resistor_SMD:R_0603_1608Metric_Pad1.05x0.95mm_HandSolder, symbol Device:R
- added TP14: TestPoint, TestPoint:TestPoint_Pad_D1.0mm, symbol Connector:TestPoint
- added U3: TPS61222DCK, Package_TO_SOT_SMD:Texas_R-PDSO-G6, symbol Regulator_Switching:TPS61222DCK
- added U5: MAX17260, Package_DFN_QFN:DFN-14-1EP_3x3mm_P0.4mm_EP1.78x2.35mm, symbol custom:MAX17260
- BT1: footprint Connector_JST:JST_SH_SM02B-SRSS-TB_1x02-1MP_P1.00mm_Horizontal -> Connector_JST:JST_PH_S2B-PH-K_1x02_P2.00mm_Horizontal
- L1: value 1uF -> 2.2uH
Connections:
- net labels added: +5V, BATTPOW
- net labels removed: BATREAD
- wire segments 203 -> 229
- no-connect marks 27 -> 30
Other:
- note added: "Regulates to 5v"
- moved on the sheet: U2
