File: kicad/watch/watch.kicad_pcb (KiCad board)
At the start: 2 copper layers, 35.6 x 25.4 mm, 55 parts, among them IC1 113990582, M41T62Q M41T62Q, Q1 DMN6140L, Q2 DMN6140L, Y1 Crystal, Y2 32.768 kHz

Commit message: un-derped pcb references
Parts:
- J1: renamed from USB C
- J2: renamed from btns 123
- J3: renamed from btns 456
- J4: renamed from Memory LCD
- JP2: renamed from 3v3 <> btn6
- U1: renamed from W25 Flash
- renumbered Schottkey to D1, frontlight to J5, buzzer to J6, BOOT to SW_BOOT1, RESET to SW_RESET1, 3v3 to TP1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
