File: kicad/watch/usbstub/usbstub/usbstub.kicad_pcb (KiCad board)
At the start: 2 copper layers, 8.5 x 17.8 mm, 6 parts, among them J1 USB_C_Receptacle_USB2.0, J2 Conn_01x04_Female

Commit message: checkpoint before retooling board...again.
Other:
- board text added: "+"
Changed lines of the file:
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@@
   (general
     (thickness 1.6)
-    (drawings 8)
+    (drawings 9)
     (tracks 53)
     (zones 0)
@@
   (page A4)
   (layers
-    (0 F.Cu signal)
+    (0 F.Cu signal hide)
     (31 B.Cu signal)
     (32 B.Adhes user)
@@
     (pad MP smd roundrect (at 2.8 -1.875 270) (size 1.2 1.8) (layers B.Cu B.Paste B.Mask) (roundrect_rratio 0.208333))
     (model /home/jeff/code/nrf52-watch/kicad/libs/jst.step
-      (offset (xyz 0 1 -0.25))
+      (offset (xyz 0 1 -0.5))
       (scale (xyz 1 1 1))
       (rotate (xyz -90 0 0))
@@
     (pad "" np_thru_hole circle (at 0 0) (size 2.1 2.1) (drill 2.1) (layers *.Cu *.Mask))
   )
+  (gr_text + (at -2.5 -1.75) (layer B.SilkS)
+    (effects (font (size 1.5 1.5) (thickness 0.3)) (justify mirror))
+  )
   (gr_line (start 0 -9) (end 4.5 -9) (layer Edge.Cuts) (width 0.15))
