File: kicad/watch/buttonpanel/buttonpanel/buttonpanel.kicad_pcb (KiCad board)
At the start: 2 copper layers, 40 x 8 mm, 4 parts, among them J1 Conn_01x04_Female, SW1 SW_Push, SW2 SW_Push, SW3 SW_Push

Commit message: pcbs ordered :)
Parts:
- SW1, SW2, SW3: footprint Button_Switch_SMD:SW_Push_1P1T_NO_6x6mm_H9.5mm -> Button_Switch_SMD:SW_SPST_CK_KXT3
Routing:
- net GND: track 0.00 -> 29.8 mm, vias 0 -> 1
- net B1: track 0.00 -> 17.8 mm, vias 0 -> 1
- net B3: track 0.00 -> 10.00 mm, vias 0 -> 1
- net B2: track 0.00 -> 4.24 mm, vias 0 -> 1
Other:
- board size 40 x 8 mm -> 33 x 8 mm
