File: kicad/watch/buttonpanel/buttonpanel/buttonpanel.sch (KiCad schematic (older format))
At the start: 4 parts, among them J1 Conn_01x04_Female, SW1 SW_Push, SW2 SW_Push, SW3 SW_Push

Commit message: pcbs ordered :)
Parts:
- SW1, SW2, SW3: footprint Button_Switch_SMD:SW_Push_1P1T_NO_6x6mm_H9.5mm -> Button_Switch_SMD:SW_SPST_CK_KXT3
Changed lines of the file:
@@
 EESchema Schematic File Version 4
+LIBS:buttonpanel-cache
 EELAYER 26 0
 EELAYER END
@@
 F 0 "SW1" H 4350 1935 50  0000 C CNN
 F 1 "SW_Push" H 4350 1844 50  0000 C CNN
-F 2 "Button_Switch_SMD:SW_Push_1P1T_NO_6x6mm_H9.5mm" H 4350 1850 50  0001 C CNN
+F 2 "Button_Switch_SMD:SW_SPST_CK_KXT3" H 4350 1850 50  0001 C CNN
 F 3 "~" H 4350 1850 50  0001 C CNN
 	1    4350 1650
@@
 F 0 "SW2" H 4350 2385 50  0000 C CNN
 F 1 "SW_Push" H 4350 2294 50  0000 C CNN
-F 2 "Button_Switch_SMD:SW_Push_1P1T_NO_6x6mm_H9.5mm" H 4350 2300 50  0001 C CNN
+F 2 "Button_Switch_SMD:SW_SPST_CK_KXT3" H 4350 2300 50  0001 C CNN
 F 3 "~" H 4350 2300 50  0001 C CNN
 	1    4350 2100
@@
 F 0 "SW3" H 4350 2885 50  0000 C CNN
 F 1 "SW_Push" H 4350 2794 50  0000 C CNN
-F 2 "Button_Switch_SMD:SW_Push_1P1T_NO_6x6mm_H9.5mm" H 4350 2800 50  0001 C CNN
+F 2 "Button_Switch_SMD:SW_SPST_CK_KXT3" H 4350 2800 50  0001 C CNN
 F 3 "~" H 4350 2800 50  0001 C CNN
 	1    4350 2600
