File: kicad/watch/watch-logic/watch-logic.kicad_pcb (KiCad board)
At the start: 2 copper layers, 25.4 x 25.4 mm, 41 parts, among them IC1 113990582, IC2 M41T62LC6F, J1 Conn_01x04_Female, J2 Conn_01x04_Female, J3 Buzzer, J4 Memory LCD, J5 Conn_01x04_Female, P1 AXT610124, Q1 DMN6140L, Q2 DMN6140L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

Commit message: snapshot for upload to github, now that copyrights are cleared
Parts:
- moved P1 3.00 mm to (170.4, 133.3)
Routing:
- net SCL: track 35.9 -> 41.5 mm
- net VBUS: track 15.4 -> 20.5 mm
- net USB_DN: track 9.99 -> 14.1 mm
- net SDA: track 43.5 -> 47.3 mm
- net USB_DP: track 10.3 -> 13.8 mm
- net GND: track 91.5 -> 94.5 mm
- net +5V: track 26.2 -> 28.7 mm
- net +3V3: track 58.5 -> 60.8 mm
