File: kicad/watch-mk2/flex/flex/_autosave-flex.kicad_pcb (KiCad board)
At the start: 2 copper layers, 33.6 x 41.5 mm, 11 parts, among them P1 AXT510124, Q1 Si1308EDL, SW1 MCSLPT4644B4PHTR, SW2 MCSLPT4644B4PHTR

Commit message: add rev2 of flex cable
Changed lines of the file:
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@@
       (drillshape 0)
       (scaleselection 1)
-      (outputdirectory "../gerber/rev2/")
+      (outputdirectory "../gerber/rev2.1/")
     )
   )
@@
     (fp_line (start -3.15 -1.6) (end 3.15 -1.6) (layer "F.Fab") (width 0.1))
     (fp_line (start -3.15 1.6) (end -3.15 -1.6) (layer "F.Fab") (width 0.1))
-    (pad "2" smd roundrect (at 2.9 0 180) (size 1.35 3.35) (layers "F.Cu" "F.Paste" "F.Mask") (roundrect_rratio 0.185185)
+    (pad "2" smd roundrect (at 2.9 0 180) (size 1.35 3.35) (layers "F.Cu" "F.Paste" "F.Mask") (roundrect_rratio 0.1851851851851852)
       (net 1 "Net-(D1-Pad2)"))
-    (pad "1" smd roundrect (at -2.9 0 180) (size 1.35 3.35) (layers "F.Cu" "F.Paste" "F.Mask") (roundrect_rratio 0.185185)
+    (pad "1" smd roundrect (at -2.9 0 180) (size 1.35 3.35) (layers "F.Cu" "F.Paste" "F.Mask") (roundrect_rratio 0.1851851851851852)
       (net 4 "VIN"))
     (model "${KISYS3DMOD}/Resistor_SMD.3dshapes/R_2512_6332Metric.wrl"
